Commit message: make gazebo runnable with the kitbot in the scene

File: src/kitbot_description/urdf/kb_25000.urdf (robot description, URDF)
Before this commit: robot kb_25000, 553 links, 552 joints
Links:
- removed link 130t_5mm_x_15mm_htd_belt__wcp_0652_
- removed link 160t_belt___800_5m_15
- removed link 160t_belt___800_5m_15_1
- removed link 160t_belt___800_5m_15_2
- removed link 160t_belt___800_5m_15_3
Joints:
- removed joint belt____pulley
- removed joint belt____pulley_1
- removed joint belt____pulley_2
- removed joint belt____pulley_3
- removed joint fixed_components_fastened_joint_58
- joint fixed_components_fastened_joint_33: child 130t_5mm_x_15mm_htd_belt__wcp_0652_ -> kb_25009

Commit message: clean kitbot joints and add joint controller gz plugins

File: src/kitbot_description/urdf/kb_25000.urdf (robot description, URDF)
Before this commit: robot kb_25000, 548 links, 547 joints
Joints:
- joint output_shaft_revolute: type continuous -> fixed
- joint output_shaft_revolute_1: type continuous -> fixed
- joint wheel_revolute_loop_closure: type continuous -> fixed
- joint wheel_revolute_loop_closure_1: type continuous -> fixed
- joint wheel_revolute_loop_closure_2: type continuous -> fixed
- joint wheel_revolute_loop_closure_3: type continuous -> fixed

Commit message: add teleop controls for kitbot

File: src/kitbot_description/urdf/kb_25000.urdf (robot description, URDF)
Before this commit: robot kb_25000, 548 links, 547 joints
Joints:
- joint wheel_revolute_2: axis -1 1.52717e-14 6.35175e-15 -> 1 1.52717e-14 6.35175e-15
- joint wheel_revolute_3: axis -1 1.52717e-14 6.35175e-15 -> 1 1.52717e-14 6.35175e-15

Commit message: change kitbot center of mass

File: src/kitbot_description/urdf/kb_25000.urdf (robot description, URDF)
Before this commit: robot kb_25000, 548 links, 547 joints
Links:
- added link ballast, mass 4.0; collision box size=0.18 0.18 0.05; visual box size=0.18 0.18 0.05
Joints:
- added joint ballast_joint: type fixed, parent root, child ballast, origin xyz=0 0 0.05 rpy=0 0 0
