Commit message: create basic kinematic tree for g2 urdf

File: src/g2_description/urdf/g2.urdf (robot description, URDF)
Before this commit: robot None, 19 links, 3 joints
Joints:
- added joint intake_right: type continuous, parent intake_end_effector, child intake_compliant_wheels_right, origin xyz=0.0 0.0 0.0 rpy=0.0 0.0 0.0, axis 0.0 0.0 0.0, limit lower=0.0 upper=0.0 effort=0.0 velocity=0.0
- added joint shooter_body: type revolute, parent shooter_dif_ring, child shooter_body, origin xyz=0.0 0.0 0.0 rpy=0.0 0.0 0.0, axis 0.0 0.0 0.0, limit lower=0.0 upper=0.0 effort=0.0 velocity=0.0
- added joint shooter_compliant_wheel_1: type continuous, parent shooter_body, child shooter_compliant_wheel_1, origin xyz=0.0 0.0 0.0 rpy=0.0 0.0 0.0, axis 0.0 0.0 0.0, limit lower=0.0 upper=0.0 effort=0.0 velocity=0.0
- added joint shooter_compliant_wheel_2: type continuous, parent shooter_body, child shooter_compliant_wheel_2, origin xyz=0.0 0.0 0.0 rpy=0.0 0.0 0.0, axis 0.0 0.0 0.0, limit lower=0.0 upper=0.0 effort=0.0 velocity=0.0
- added joint shooter_compliant_wheel_3: type continuous, parent shooter_body, child shooter_compliant_wheel_3, origin xyz=0.0 0.0 0.0 rpy=0.0 0.0 0.0, axis 0.0 0.0 0.0, limit lower=0.0 upper=0.0 effort=0.0 velocity=0.0
- added joint shooter_compliant_wheel_feeder: type continuous, parent shooter_body, child shooter_compliant_wheel_feeder, origin xyz=0.0 0.0 0.0 rpy=0.0 0.0 0.0, axis 0.0 0.0 0.0, limit lower=0.0 upper=0.0 effort=0.0 velocity=0.0
- added joint shooter_dif_ring: type revolute, parent chassis, child shooter_dif_ring, origin xyz=0.0 0.0 0.0 rpy=0.0 0.0 0.0, axis 0.0 0.0 0.0, limit lower=0.0 upper=0.0 effort=0.0 velocity=0.0
- added joint swerve_axel_back_left: type continuous, parent chassis, child swerve_axel_back_left, origin xyz=0.0 0.0 0.0 rpy=0.0 0.0 0.0, axis 0.0 0.0 0.0, limit lower=0.0 upper=0.0 effort=0.0 velocity=0.0
- added joint swerve_axel_back_right: type continuous, parent chassis, child swerve_axel_back_right, origin xyz=0.0 0.0 0.0 rpy=0.0 0.0 0.0, axis 0.0 0.0 0.0, limit lower=0.0 upper=0.0 effort=0.0 velocity=0.0
- added joint swerve_axel_front_left: type continuous, parent chassis, child swerve_axel_front_left, origin xyz=0.0 0.0 0.0 rpy=0.0 0.0 0.0, axis 0.0 0.0 0.0, limit lower=0.0 upper=0.0 effort=0.0 velocity=0.0
- added joint swerve_axel_front_right: type continuous, parent chassis, child swerve_axel_front_right, origin xyz=0.0 0.0 0.0 rpy=0.0 0.0 0.0, axis 0.0 0.0 0.0, limit lower=0.0 upper=0.0 effort=0.0 velocity=0.0
- added joint swerve_wheel_back_left: type continuous, parent swerve_axel_back_left, child swerve_wheel_back_left, origin xyz=0.0 0.0 0.0 rpy=0.0 0.0 0.0, axis 0.0 0.0 0.0, limit lower=0.0 upper=0.0 effort=0.0 velocity=0.0
- added joint swerve_wheel_back_right: type continuous, parent swerve_axel_back_right, child swerve_wheel_back_right, origin xyz=0.0 0.0 0.0 rpy=0.0 0.0 0.0, axis 0.0 0.0 0.0, limit lower=0.0 upper=0.0 effort=0.0 velocity=0.0
- added joint swerve_wheel_front_left: type continuous, parent swerve_axel_front_left, child swerve_wheel_front_left, origin xyz=0.0 0.0 0.0 rpy=0.0 0.0 0.0, axis 0.0 0.0 0.0, limit lower=0.0 upper=0.0 effort=0.0 velocity=0.0
- added joint swerve_wheel_front_right: type continuous, parent swerve_axel_front_right, child swerve_wheel_front_right, origin xyz=0.0 0.0 0.0 rpy=0.0 0.0 0.0, axis 0.0 0.0 0.0, limit lower=0.0 upper=0.0 effort=0.0 velocity=0.0

Commit message: add meshes, chassis mesh to the urdf, add rviz launch script

File: src/g2_description/urdf/g2.urdf (robot description, URDF)
Before this commit: robot g2_2025, 19 links, 18 joints
Links:
- link chassis: geometry visual mesh filename=package://g2_description/meshes/Chassis.dae scale=1 1 1

Commit message: add tuner stuff

File: src/g2_description/urdf/g2.urdf (robot description, URDF)
Before this commit: robot g2_2025, 19 links, 18 joints
Links:
- link intake: geometry visual mesh filename=package://g2_description/meshes/Intake.dae
- link intake_compliant_wheels_left: geometry visual mesh filename=package://g2_description/meshes/Intake Compliant Wheel Stac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
- link intake_compliant_wheels_right: geometry visual mesh filename=package://g2_description/meshes/Intake Compliant Wheel Stac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
- link intake_end_effector: geometry visual mesh filename=package://g2_description/meshes/Intake End Effector.dae
- link shooter_body: geometry visual mesh filename=package://g2_description/meshes/Shooter Body.dae
- link shooter_compliant_wheel_1: geometry visual mesh filename=package://g2_description/meshes/Shooter Compliant Wheel.dae
- link shooter_compliant_wheel_2: geometry visual mesh filename=package://g2_description/meshes/Shooter Compliant Wheel.dae
- link shooter_compliant_wheel_3: geometry visual mesh filename=package://g2_description/meshes/Shooter Compliant Wheel.dae
- link shooter_compliant_wheel_feeder: geometry visual mesh filename=package://g2_description/meshes/Shooter Compliant Wheel.dae
- link shooter_dif_ring: geometry visual mesh filename=package://g2_description/meshes/Dif Ring.dae
- link swerve_axel_back_left: geometry visual mesh filename=package://g2_description/meshes/Swerve Axel.dae
- link swerve_axel_back_right: geometry visual mesh filename=package://g2_description/meshes/Swerve Axel.dae
- link swerve_axel_front_left: geometry visual mesh filename=package://g2_description/meshes/Swerve Axel.dae
- link swerve_axel_front_right: geometry visual mesh filename=package://g2_description/meshes/Swerve Axel.dae
- link swerve_wheel_back_left: geometry visual mesh filename=package://g2_description/meshes/Swerve Wheel.dae
- link swerve_wheel_back_right: geometry visual mesh filename=package://g2_description/meshes/Swerve Wheel.dae
- link swerve_wheel_front_left: geometry visual mesh filename=package://g2_description/meshes/Swerve Wheel.dae
- link swerve_wheel_front_right: geometry visual mesh filename=package://g2_description/meshes/Swerve Wheel.dae

Commit message: add offset for prismatic joint

File: src/g2_description/urdf/g2.urdf (robot description, URDF)
Before this commit: robot g2_2025, 19 links, 18 joints
Joints:
- joint linear_actuators: axis 0.0 0.0 0.0 -> 0.0 1 0.0; origin xyz=0.0 0.0 0.0 rpy=0.0 0.0 0.0 -> xyz=0.0 -0.341 0.038 rpy=0.0 0.0 0.0

Commit message: create usable urdf for g2; add some tooling for creating urdf

File: src/g2_description/urdf/g2.urdf (robot description, URDF)
Before this commit: robot g2_2025, 19 links, 18 joints
Joints:
- joint intake_left: axis 0.0 0.0 0.0 -> 0.0 0.0 1; origin xyz=0.0 0.0 0.0 rpy=0.0 0.0 0.0 -> xyz=0.095 -0.119 -0.11 rpy=0.0 0.0 0.0
- joint intake_pivot: axis 0.0 0.0 0.0 -> 1 0.0 0.0; origin xyz=0.0 0.0 0.0 rpy=0.0 0.0 0.0 -> xyz=0.0 -0.13 0.031 rpy=0.0 0.0 0.0
- joint intake_right: axis 0.0 0.0 0.0 -> 0.0 0.0 1; origin xyz=0.0 0.0 0.0 rpy=0.0 0.0 0.0 -> xyz=-0.095 -0.119 -0.11 rpy=0.0 0.0 0.0
- joint shooter_body: axis 0.0 0.0 0.0 -> 1 0.0 0.0; origin xyz=0.0 0.0 0.0 rpy=0.0 0.0 0.0 -> xyz=0.0 0.0 0.03 rpy=0.0 0.0 0.479965544
- joint shooter_compliant_wheel_1: axis 0.0 0.0 0.0 -> 0.0 1 0.0; origin xyz=0.0 0.0 0.0 rpy=0.0 0.0 0.0 -> xyz=0.0 -0.352 0.245 rpy=0.0 0.0 1.57079633
- joint shooter_compliant_wheel_2: axis 0.0 0.0 0.0 -> 1 0.0 0.0; origin xyz=0.0 0.0 0.0 rpy=0.0 0.0 0.0 -> xyz=0.068 -0.351 0.064 rpy=0.0 -0.785398163 0.0
- joint shooter_compliant_wheel_3: axis 0.0 0.0 0.0 -> 0.0 1 0.0; origin xyz=0.0 0.0 0.0 rpy=0.0 0.0 0.0 -> xyz=-0.078 -0.352 0.067 rpy=-2.35619449 0.0 1.57079633
- joint shooter_compliant_wheel_feeder: axis 0.0 0.0 0.0 -> 0.0 1 0.0; origin xyz=0.0 0.0 0.0 rpy=0.0 0.0 0.0 -> xyz=0.0 -0.035 0.245 rpy=0.0 0.0 1.57079633
- joint shooter_dif_ring: axis 0.0 0.0 0.0 -> 0.0 0.0 1; origin xyz=0.0 0.0 0.0 rpy=0.0 0.0 0.0 -> xyz=0.0 0.274 0.024 rpy=0.0 0.0 -0.479965544
- joint swerve_axel_back_left: axis 0.0 0.0 0.0 -> 0.0 0.0 1; origin xyz=0.0 0.0 0.0 rpy=0.0 0.0 0.0 -> xyz=0.264 0.364 -0.088 rpy=0.0 0.0 0.0
- joint swerve_axel_back_right: axis 0.0 0.0 0.0 -> 0.0 0.0 1; origin xyz=0.0 0.0 0.0 rpy=0.0 0.0 0.0 -> xyz=-0.238 0.364 -0.088 rpy=0.0 0.0 0.0
- joint swerve_axel_front_left: axis 0.0 0.0 0.0 -> 0.0 0.0 1; origin xyz=0.0 0.0 0.0 rpy=0.0 0.0 0.0 -> xyz=0.264 -0.364 -0.088 rpy=0.0 0.0 0.0
- joint swerve_axel_front_right: axis 0.0 0.0 0.0 -> 0.0 0.0 1; origin xyz=0.0 0.0 0.0 rpy=0.0 0.0 0.0 -> xyz=-0.264 -0.364 -0.088 rpy=0.0 0.0 0.0
- joint swerve_wheel_back_left: axis 0.0 0.0 0.0 -> 0.0 1 0.0; origin xyz=0.0 0.0 0.0 rpy=0.0 0.0 0.0 -> xyz=0.002 0.0 -0.023 rpy=0.0 0.0 0.0
- joint swerve_wheel_back_right: axis 0.0 0.0 0.0 -> 0.0 1 0.0; origin xyz=0.0 0.0 0.0 rpy=0.0 0.0 0.0 -> xyz=0.002 0.0 -0.023 rpy=0.0 0.0 0.0
- joint swerve_wheel_front_left: axis 0.0 0.0 0.0 -> 0.0 1 0.0; origin xyz=0.0 0.0 0.0 rpy=0.0 0.0 0.0 -> xyz=0.002 0.0 -0.023 rpy=0.0 0.0 0.0
- joint swerve_wheel_front_right: axis 0.0 0.0 0.0 -> 0.0 1 0.0; origin xyz=0.0 0.0 0.0 rpy=0.0 0.0 0.0 -> xyz=0.002 0.0 -0.023 rpy=0.0 0.0 0.0

Commit message: get in running in gazebo fully

File: src/g2_description/urdf/g2.urdf (robot description, URDF)
Before this commit: robot g2_2025, 19 links, 18 joints
Links:
- link chassis: mass None -> 25; geometry collision mesh filename=package://g2_description/meshes/collision/Chassis.stl scale=1 1 1; visual mesh filename=package://g2_description/meshes/visual/Chassis.glb scale=1 1 1
- link intake: mass None -> 3; geometry collision mesh filename=package://g2_description/meshes/collision/Intake.stl; visual mesh filename=package://g2_description/meshes/visual/Intake.glb
- link intake_compliant_wheels_left: mass None -> 0.3; geometry collision mesh filename=package://g2_description/meshes/collision/Intake_Compliant_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; visual mesh filename=package://g2_description/meshes/visual/Intake_Compliant_Whe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
- link intake_compliant_wheels_right: mass None -> 0.3; geometry collision mesh filename=package://g2_description/meshes/collision/Intake_Compliant_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; visual mesh filename=package://g2_description/meshes/visual/Intake_Compliant_Whe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
- link intake_end_effector: mass None -> 1.5; geometry collision mesh filename=package://g2_description/meshes/collision/Intake_End_Effect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; visual mesh filename=package://g2_description/meshes/visual/Intake_End_Effector.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
- link shooter_body: mass None -> 4; geometry collision mesh filename=package://g2_description/meshes/collision/Shooter_Body.stl; visual mesh filename=package://g2_description/meshes/visual/Shooter_Body.glb
- link shooter_compliant_wheel_1: mass None -> 0.25; geometry collision mesh filename=package://g2_description/meshes/collision/Shooter_Compliant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; visual mesh filename=package://g2_description/meshes/visual/Shooter_Compliant_Wh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
- link shooter_compliant_wheel_2: mass None -> 0.25; geometry collision mesh filename=package://g2_description/meshes/collision/Shooter_Compliant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; visual mesh filename=package://g2_description/meshes/visual/Shooter_Compliant_Wh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
- link shooter_compliant_wheel_3: mass None -> 0.25; geometry collision mesh filename=package://g2_description/meshes/collision/Shooter_Compliant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; visual mesh filename=package://g2_description/meshes/visual/Shooter_Compliant_Wh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
- link shooter_compliant_wheel_feeder: mass None -> 0.25; geometry collision mesh filename=package://g2_description/meshes/collision/Shooter_Compliant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; visual mesh filename=package://g2_description/meshes/visual/Shooter_Compliant_Wh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
- link shooter_dif_ring: mass None -> 1; geometry collision mesh filename=package://g2_description/meshes/collision/Dif_Ring.stl; visual mesh filename=package://g2_description/meshes/visual/Dif_Ring.glb
- link swerve_axel_back_left: mass None -> 1.5; geometry collision mesh filename=package://g2_description/meshes/collision/Swerve_Axel.stl; visual mesh filename=package://g2_description/meshes/visual/Swerve_Axel.glb
- link swerve_axel_back_right: mass None -> 1.5; geometry collision mesh filename=package://g2_description/meshes/collision/Swerve_Axel.stl; visual mesh filename=package://g2_description/meshes/visual/Swerve_Axel.glb
- link swerve_axel_front_left: mass None -> 1.5; geometry collision mesh filename=package://g2_description/meshes/collision/Swerve_Axel.stl; visual mesh filename=package://g2_description/meshes/visual/Swerve_Axel.glb
- link swerve_axel_front_right: mass None -> 1.5; geometry collision mesh filename=package://g2_description/meshes/collision/Swerve_Axel.stl; visual mesh filename=package://g2_description/meshes/visual/Swerve_Axel.glb
- link swerve_wheel_back_left: mass None -> 0.6; geometry collision mesh filename=package://g2_description/meshes/collision/Swerve_Wheel.stl; visual mesh filename=package://g2_description/meshes/visual/Swerve_Wheel.glb
- link swerve_wheel_back_right: mass None -> 0.6; geometry collision mesh filename=package://g2_description/meshes/collision/Swerve_Wheel.stl; visual mesh filename=package://g2_description/meshes/visual/Swerve_Wheel.glb
- link swerve_wheel_front_left: mass None -> 0.6; geometry collision mesh filename=package://g2_description/meshes/collision/Swerve_Wheel.stl; visual mesh filename=package://g2_description/meshes/visual/Swerve_Wheel.glb
- link swerve_wheel_front_right: mass None -> 0.6; geometry collision mesh filename=package://g2_description/meshes/collision/Swerve_Wheel.stl; visual mesh filename=package://g2_description/meshes/visual/Swerve_Wheel.glb
Joints:
- removed joint shooter_body
- removed joint shooter_compliant_wheel_1
- removed joint shooter_compliant_wheel_2
- removed joint shooter_compliant_wheel_3
- removed joint shooter_compliant_wheel_feeder
- removed joint shooter_dif_ring
- removed joint swerve_axel_back_left
- removed joint swerve_axel_back_right
- removed joint swerve_axel_front_left
- removed joint swerve_axel_front_right
- removed joint swerve_wheel_back_left
- removed joint swerve_wheel_back_right
- removed joint swerve_wheel_front_left
- removed joint swerve_wheel_front_right
- added joint shooter_body_joint: type revolute, parent shooter_dif_ring, child shooter_body, origin xyz=0.0 0.0 0.03 rpy=0.0 0.0 0.479965544, axis 1 0.0 0.0, limit lower=0.0 upper=0.0 effort=0.0 velocity=0.0
- added joint shooter_compliant_wheel_1_joint: type continuous, parent shooter_body, child shooter_compliant_wheel_1, origin xyz=0.0 -0.352 0.245 rpy=0.0 0.0 1.57079633, axis 0.0 1 0.0, limit lower=0.0 upper=0.0 effort=0.0 velocity=0.0
- added joint shooter_compliant_wheel_2_joint: type continuous, parent shooter_body, child shooter_compliant_wheel_2, origin xyz=0.068 -0.351 0.064 rpy=0.0 -0.785398163 0.0, axis 1 0.0 0.0, limit lower=0.0 upper=0.0 effort=0.0 velocity=0.0
- added joint shooter_compliant_wheel_3_joint: type continuous, parent shooter_body, child shooter_compliant_wheel_3, origin xyz=-0.078 -0.352 0.067 rpy=-2.35619449 0.0 1.57079633, axis 0.0 1 0.0, limit lower=0.0 upper=0.0 effort=0.0 velocity=0.0
- added joint shooter_compliant_wheel_feeder_joint: type continuous, parent shooter_body, child shooter_compliant_wheel_feeder, origin xyz=0.0 -0.035 0.245 rpy=0.0 0.0 1.57079633, axis 0.0 1 0.0, limit lower=0.0 upper=0.0 effort=0.0 velocity=0.0
- added joint shooter_dif_ring_joint: type revolute, parent chassis, child shooter_dif_ring, origin xyz=0.0 0.274 0.024 rpy=0.0 0.0 -0.479965544, axis 0.0 0.0 1, limit lower=0.0 upper=0.0 effort=0.0 velocity=0.0
- added joint swerve_axel_back_left_joint: type continuous, parent chassis, child swerve_axel_back_left, origin xyz=0.264 0.364 -0.088 rpy=0.0 0.0 0.0, axis 0.0 0.0 1, limit lower=0.0 upper=0.0 effort=0.0 velocity=0.0
- added joint swerve_axel_back_right_joint: type continuous, parent chassis, child swerve_axel_back_right, origin xyz=-0.238 0.364 -0.088 rpy=0.0 0.0 0.0, axis 0.0 0.0 1, limit lower=0.0 upper=0.0 effort=0.0 velocity=0.0
- added joint swerve_axel_front_left_joint: type continuous, parent chassis, child swerve_axel_front_left, origin xyz=0.264 -0.364 -0.088 rpy=0.0 0.0 0.0, axis 0.0 0.0 1, limit lower=0.0 upper=0.0 effort=0.0 velocity=0.0
- added joint swerve_axel_front_right_joint: type continuous, parent chassis, child swerve_axel_front_right, origin xyz=-0.264 -0.364 -0.088 rpy=0.0 0.0 0.0, axis 0.0 0.0 1, limit lower=0.0 upper=0.0 effort=0.0 velocity=0.0
- added joint swerve_wheel_back_left_joint: type continuous, parent swerve_axel_back_left, child swerve_wheel_back_left, origin xyz=0.002 0.0 -0.023 rpy=0.0 0.0 0.0, axis 0.0 1 0.0, limit lower=0.0 upper=0.0 effort=0.0 velocity=0.0
- added joint swerve_wheel_back_right_joint: type continuous, parent swerve_axel_back_right, child swerve_wheel_back_right, origin xyz=0.002 0.0 -0.023 rpy=0.0 0.0 0.0, axis 0.0 1 0.0, limit lower=0.0 upper=0.0 effort=0.0 velocity=0.0
- added joint swerve_wheel_front_left_joint: type continuous, parent swerve_axel_front_left, child swerve_wheel_front_left, origin xyz=0.002 0.0 -0.023 rpy=0.0 0.0 0.0, axis 0.0 1 0.0, limit lower=0.0 upper=0.0 effort=0.0 velocity=0.0
- added joint swerve_wheel_front_right_joint: type continuous, parent swerve_axel_front_right, child swerve_wheel_front_right, origin xyz=0.002 0.0 -0.023 rpy=0.0 0.0 0.0, axis 0.0 1 0.0, limit lower=0.0 upper=0.0 effort=0.0 velocity=0.0
