Commit message: refactor to remove the g2_ prefix

File: src/description/urdf/g2.urdf (robot description, URDF)
Before this commit: robot g2_2025, 19 links, 18 joints
Links:
- link chassis: geometry collision mesh filename=package://description/meshes/collision/Chassis.stl scale=1 1 1; visual mesh filename=package://description/meshes/visual/Chassis.glb scale=1 1 1
- link intake: geometry collision mesh filename=package://description/meshes/collision/Intake.stl; visual mesh filename=package://description/meshes/visual/Intake.glb
- link intake_compliant_wheels_left: geometry collision mesh filename=package://description/meshes/collision/Intake_Compliant_Whe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; visual mesh filename=package://description/meshes/visual/Intake_Compliant_Wheel_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
- link intake_compliant_wheels_right: geometry collision mesh filename=package://description/meshes/collision/Intake_Compliant_Whe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; visual mesh filename=package://description/meshes/visual/Intake_Compliant_Wheel_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
- link intake_end_effector: geometry collision mesh filename=package://description/meshes/collision/Intake_End_Effector.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; visual mesh filename=package://description/meshes/visual/Intake_End_Effector.glb
- link shooter_body: geometry collision mesh filename=package://description/meshes/collision/Shooter_Body.stl; visual mesh filename=package://description/meshes/visual/Shooter_Body.glb
- link shooter_compliant_wheel_1: geometry collision mesh filename=package://description/meshes/collision/Shooter_Compliant_Wh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; visual mesh filename=package://description/meshes/visual/Shooter_Compliant_Wheel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
- link shooter_compliant_wheel_2: geometry collision mesh filename=package://description/meshes/collision/Shooter_Compliant_Wh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; visual mesh filename=package://description/meshes/visual/Shooter_Compliant_Wheel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
- link shooter_compliant_wheel_3: geometry collision mesh filename=package://description/meshes/collision/Shooter_Compliant_Wh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; visual mesh filename=package://description/meshes/visual/Shooter_Compliant_Wheel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
- link shooter_compliant_wheel_feeder: geometry collision mesh filename=package://description/meshes/collision/Shooter_Compliant_Wh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; visual mesh filename=package://description/meshes/visual/Shooter_Compliant_Wheel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
- link shooter_dif_ring: geometry collision mesh filename=package://description/meshes/collision/Dif_Ring.stl; visual mesh filename=package://description/meshes/visual/Dif_Ring.glb
- link swerve_axel_back_left: geometry collision mesh filename=package://description/meshes/collision/Swerve_Axel.stl; visual mesh filename=package://description/meshes/visual/Swerve_Axel.glb
- link swerve_axel_back_right: geometry collision mesh filename=package://description/meshes/collision/Swerve_Axel.stl; visual mesh filename=package://description/meshes/visual/Swerve_Axel.glb
- link swerve_axel_front_left: geometry collision mesh filename=package://description/meshes/collision/Swerve_Axel.stl; visual mesh filename=package://description/meshes/visual/Swerve_Axel.glb
- link swerve_axel_front_right: geometry collision mesh filename=package://description/meshes/collision/Swerve_Axel.stl; visual mesh filename=package://description/meshes/visual/Swerve_Axel.glb
- link swerve_wheel_back_left: geometry collision mesh filename=package://description/meshes/collision/Swerve_Wheel.stl; visual mesh filename=package://description/meshes/visual/Swerve_Wheel.glb
- link swerve_wheel_back_right: geometry collision mesh filename=package://description/meshes/collision/Swerve_Wheel.stl; visual mesh filename=package://description/meshes/visual/Swerve_Wheel.glb
- link swerve_wheel_front_left: geometry collision mesh filename=package://description/meshes/collision/Swerve_Wheel.stl; visual mesh filename=package://description/meshes/visual/Swerve_Wheel.glb
- link swerve_wheel_front_right: geometry collision mesh filename=package://description/meshes/collision/Swerve_Wheel.stl; visual mesh filename=package://description/meshes/visual/Swerve_Wheel.glb

Commit message: add motor simulation node

File: src/description/urdf/g2.urdf (robot description, URDF)
Before this commit: robot g2_2025, 19 links, 18 joints
Joints:
- joint swerve_axel_back_left_joint: limit lower=0.0 upper=0.0 effort=0.0 velocity=0.0 -> lower=0.0 upper=0.0 effort=59.3 velocity=89.4
- joint swerve_axel_back_right_joint: limit lower=0.0 upper=0.0 effort=0.0 velocity=0.0 -> lower=0.0 upper=0.0 effort=59.3 velocity=89.4
- joint swerve_axel_front_left_joint: limit lower=0.0 upper=0.0 effort=0.0 velocity=0.0 -> lower=0.0 upper=0.0 effort=59.3 velocity=89.4
- joint swerve_axel_front_right_joint: limit lower=0.0 upper=0.0 effort=0.0 velocity=0.0 -> lower=0.0 upper=0.0 effort=59.3 velocity=89.4
- joint swerve_wheel_back_left_joint: limit lower=0.0 upper=0.0 effort=0.0 velocity=0.0 -> lower=0.0 upper=0.0 effort=59.3 velocity=89.4
- joint swerve_wheel_back_right_joint: limit lower=0.0 upper=0.0 effort=0.0 velocity=0.0 -> lower=0.0 upper=0.0 effort=59.3 velocity=89.4
- joint swerve_wheel_front_left_joint: limit lower=0.0 upper=0.0 effort=0.0 velocity=0.0 -> lower=0.0 upper=0.0 effort=59.3 velocity=89.4
- joint swerve_wheel_front_right_joint: limit lower=0.0 upper=0.0 effort=0.0 velocity=0.0 -> lower=0.0 upper=0.0 effort=59.3 velocity=89.4
